Commit message: description files

File: src/carbon_description/urdf/carbon.urdf.xacro (robot description, xacro)
@@ -4,4 +4,6 @@
 	<xacro:property name="rotate90CCW" value="${3.14159 / 2}"/>
 	<xacro:property name="rotate90CW" value="${-3.14159 / 2}"/>
+	<xacro:property name="wheel_radius" value="0.09" />
+	<xacro:property name="wheel_length" value="0.0508" />
 	<xacro:property name="base_x_size" value="0.7556"/>
 	<xacro:property name="base_y_size" value="0.4572"/>
@@ -10,3 +12,6 @@
 	<xacro:include filename="$(find titan_description)/urdf/macros.xacro" />
 	<xacro:include filename="$(find titan_description)/urdf/wheel.xacro" />
+	<link name="base_link">
+		<xacro:make_box x="0.0" y="0.0" z="0.0" roll="0" pitch="0" yaw="0" sizex="${base_x_size}" sizey="${base_y_size}" sizez="${base_z_size}"/>
+	</link>
 </robot>

File: src/carbon_description/urdf/macros.xacro (robot description, xacro)
@@ -1,4 +1,4 @@
 <?xml version='1.0'?>
-<robot name="titan" xmlns:xacro="http://ros.org/wiki/xacro">
+<robot name="carbon" xmlns:xacro="http://ros.org/wiki/xacro">
 	<xacro:macro name="default_inertial" params="mass">
 		<inertial>

File: src/carbon_description/urdf/wheel.xacro (robot description, xacro)
@@ -1,4 +1,5 @@
-<robot xmlns:xacro="http://ros.org/wiki/xacro" name="titan_wheel">
-	<xacro:macro name="titan_wheel" params="wheel_prefix *joint_pose">
+<?xml version='1.0'?>
+<robot xmlns:xacro="http://ros.org/wiki/xacro" name="carbon">
+	<xacro:macro name="create_wheel" params="wheel_prefix *joint_pose">
 		<link name="${wheel_prefix}_wheel_link">
 			<inertial>

Commit message: gazebo updates

File: src/carbon_description/urdf/carbon.urdf.xacro (robot description, xacro)
@@ -1,8 +1,8 @@
 <?xml version='1.0'?>
-<robot name="carbon" xmlns:xacro="http://www.ros.org/wiki/xacro">
+<robot name="carbon" xmlns:xacro="http://ros.org/wiki/xacro">
 	<xacro:property name="M_PI" value="3.14159"/>
 	<xacro:property name="rotate90CCW" value="${3.14159 / 2}"/>
 	<xacro:property name="rotate90CW" value="${-3.14159 / 2}"/>
-	<xacro:property name="wheel_radius" value="0.09" />
+	<xacro:property name="wheel_radius" value="0.097155" />
 	<xacro:property name="wheel_length" value="0.0508" />
 	<xacro:property name="base_x_size" value="0.7556"/>
@@ -10,8 +10,81 @@
 	<xacro:property name="base_z_size" value="0.0508"/>
 	<xacro:property name="base_mass" value="10"/>
-	<xacro:include filename="$(find titan_description)/urdf/macros.xacro" />
-	<xacro:include filename="$(find titan_description)/urdf/wheel.xacro" />
+	<xacro:property name="wheelbase" value="0.58" />
+	<xacro:property name="track" value="0.25" />
+	<xacro:property name="wheel_vertical_offset" value="0.0" />
+	<xacro:arg name="robot_namespace" default="/" />
+	<xacro:include filename="$(find carbon_description)/urdf/macros.xacro" />
+	<xacro:include filename="$(find carbon_description)/urdf/wheel.xacro" />
+	<xacro:include filename="$(find carbon_description)/urdf/sick_tim.urdf.xacro" />
 	<link name="base_link">
-		<xacro:make_box x="0.0" y="0.0" z="0.0" roll="0" pitch="0" yaw="0" sizex="${base_x_size}" sizey="${base_y_size}" sizez="${base_z_size}"/>
+		<collision name='collision'>
+			<origin xyz="0 0 0" rpy="0 0 0" />
+			<geometry>
+				<box size="${base_x_size} ${base_y_size} ${base_z_size}"/>
+			</geometry>
+		</collision>
+		<visual name='base_solid'>
+			<origin xyz="0 0 0" rpy="0 0 0" />
+			<geometry>
+				<box size="${base_x_size} ${base_y_size} ${base_z_size}"/>
+			</geometry>
+			<material name="white"/>
+		</visual>
 	</link>
+	<link name="base_inertia_link">
+		<inertial>
+			<mass value="${base_mass}" />
+			<origin xyz="0 0 0" rpy=" 0 0 0"/>
+			<xacro:box_inertia m="${base_mass}" x="${base_x_size}" y="${base_y_size}" z="${base_z_size}" />
+		</inertial>
+	</link>
+	<xacro:sick_tim551 name="laser" ros_topic="scan" />
+	<joint name="base_to_inertia" type="fixed">
+		<parent link="base_link"/>
+		<child link="base_inertia_link"/>
+		<origin xyz="0 0 0" rpy="0 0 0" />
+	</joint>
+	<joint name="base_to_laser" type="fixed">
+		<parent link="base_link"/>
+		<child link="laser_mount_link"/>
+		<origin xyz="0.31 0.0 0.08" rpy="0 0 0" />
+	</joint>
+	<xacro:create_wheel wheel_prefix="left_front">
+		<origin xyz="${track} ${wheelbase/2} ${wheel_vertical_offset}" rpy="0 0 0" />
+	</xacro:create_wheel>
+	<xacro:create_wheel wheel_prefix="left_mid">
+                <origin xyz="0 ${wheelbase/2} ${wheel_vertical_offset}" rpy="0 0 0" />
+        </xacro:create_wheel>
+	<xacro:create_wheel wheel_prefix="left_rear">
+		<origin xyz="${-track} ${wheelbase/2} ${wheel_vertical_offset}" rpy="0 0 0" />
+	</xacro:create_wheel>
+	<xacro:create_wheel wheel_prefix="right_front">
+		<origin xyz="${track} ${-wheelbase/2} ${wheel_vertical_offset}" rpy="0 0 0" />
+	</xacro:create_wheel>
+	<xacro:create_wheel wheel_prefix="right_mid">
+                <origin xyz="0 ${-wheelbase/2} ${wheel_vertical_offset}" rpy="0 0 0" />
+        </xacro:create_wheel>
+	<xacro:create_wheel wheel_prefix="right_rear">
+		<origin xyz="${-track} ${-wheelbase/2} ${wheel_vertical_offset}" rpy="0 0 0" />
+	</xacro:create_wheel>
+	<gazebo>
+		<plugin name="gazebo_ros_control" filename="libgazebo_ros_control.so">
+			<robotNamespace>$(arg robot_namespace)</robotNamespace>
+		</plugin>
+	</gazebo>
+	<gazebo>
+		<plugin name="diff_drive_6w" filename="libdiffdrive_plugin_6w.so">
+			<robotNamespace>$(arg robot_namespace)</robotNamespace>
+			<topicName>/cmd_vel</topicName>
+			<frontLeftJoint>left_front_wheel</frontLeftJoint>
+			<midLeftJoint>left_mid_wheel</midLeftJoint>
+			<rearLeftJoint>left_rear_wheel</rearLeftJoint>
+			<frontRightJoint>right_front_wheel</frontRightJoint>
+			<midRightJoint>right_mid_wheel</midRightJoint>
+			<rearRightJoint>right_rear_wheel</rearRightJoint>
+			<wheelSeparation>0.58</wheelSeparation>
+			<wheelDiameter>0.18</wheelDiameter>
+			<torque>50000</torque>
+		</plugin>
+	</gazebo>
 </robot>

File: src/carbon_description/urdf/wheel.xacro (robot description, xacro)
@@ -4,13 +4,13 @@
 		<link name="${wheel_prefix}_wheel_link">
 			<inertial>
-				<mass value="5" />
+				<mass value="0.5" />
 				<!-- <inertia ixx="0.1" ixy="0.0" ixz="0.0" iyy="0.1" iyz="0.0" izz="0.1" /> -->
-				<xacro:cylinder_inertia m="1" r="${wheel_radius}" h="${wheel_length}" />
+				<xacro:cylinder_inertia m="0.5" r="${wheel_radius}" h="${wheel_length}" />
 			</inertial>
 			<visual>
-				<origin xyz="0 0 0" rpy="${M_PI/2} 0 0" />
+				<origin xyz="${wheel_radius} ${-wheel_length/2} ${-wheel_radius}" rpy="0 0 ${M_PI/2}" />
 				<geometry>
-					<!-- <mesh filename="package://titan_description/meshes/Wheel.dae" scale="0.001 0.001 0.001"/> -->
-					<cylinder length="${wheel_length}" radius="${wheel_radius}" />
+					<mesh filename="package://carbon_description/meshes/wheel.dae" scale="1.0 1.0 1.0"/>
+					<!-- <cylinder length="${wheel_length}" radius="${wheel_radius}" /> -->
 				</geometry>
 			</visual>
@@ -43,5 +43,5 @@
 			</actuator>
 			<joint name="${wheel_prefix}_wheel">
-				<hardwareInterface>hardware_interface/VelocityJointInterface</hardwareInterface>
+				<hardwareInterface>EffortJointInterface</hardwareInterface>
 			</joint>
 		</transmission>

Commit message: gazebo updates

File: src/carbon_description/urdf/carbon.urdf.xacro (robot description, xacro)
@@ -39,4 +39,15 @@
 		</inertial>
 	</link>
+	<link name="imu_link">
+		<visual name='imu_box'>
+			<origin xyz="0 0 0" rpy="0 0 0"/>
+			<geometry>
+				<box size="0.02 0.02 0.02"/>
+			</geometry>
+			<material name="green"/>
+		</visual>
+	</link>
+	<gazebo reference="imu_link">
+  	</gazebo>
 	<xacro:sick_tim551 name="laser" ros_topic="scan" />
 	<joint name="base_to_inertia" type="fixed">
@@ -49,4 +60,9 @@
 		<child link="laser_mount_link"/>
 		<origin xyz="0.31 0.0 0.08" rpy="0 0 0" />
+	</joint>
+	<joint name="base_to_imu" type="fixed">
+		<parent link="base_link"/>
+		<child link="imu_link"/>
+		<origin xyz="0 0 0" rpy="0 0 0"/>
 	</joint>
 	<xacro:create_wheel wheel_prefix="left_front">
@@ -76,5 +92,5 @@
 		<plugin name="diff_drive_6w" filename="libdiffdrive_plugin_6w.so">
 			<robotNamespace>$(arg robot_namespace)</robotNamespace>
-			<topicName>/cmd_vel</topicName>
+			<topicName>/carbon_velocity_controller/cmd_vel</topicName>
 			<frontLeftJoint>left_front_wheel</frontLeftJoint>
 			<midLeftJoint>left_mid_wheel</midLeftJoint>
@@ -88,3 +104,44 @@
 		</plugin>
 	</gazebo>
+	<!-- <gazebo>
+		<plugin name="diffdrive_plugin_multiwheel" filename="libdiffdrive_plugin_multi_wheel.so">
+			<alwaysOn>true</alwaysOn>
+			<updateRate>25.0</updateRate>
+			<leftJoints>left_front_wheel left_mid_wheel left_rear_wheel</leftJoints>
+			<rightJoints>right_front_wheel right_mid_wheel right_rear_wheel</rightJoints>
+			<wheelSeparation>${wheelbase}</wheelSeparation>
+			<wheelDiameter>${wheel_radius*2}</wheelDiameter>
+			<torque>50000</torque>
+			<robotNamespace>/</robotNamespace>
+			<robotBaseFrame>base_link</robotBaseFrame>
+			<commandTopic>/cmd_vel_raw</commandTopic>
+			<publishOdometryTf>0</publishOdometryTf>
+			<publishOdometryMsg>1</publishOdometryMsg>
+		</plugin>
+	</gazebo> -->
+	<!-- <gazebo>
+		<plugin name="force_based_move_controller" filename="libgazebo_ros_force_based_move.so">
+			<commandTopic>/carbon_velocity_controller/cmd_vel</commandTopic>
+			<odometryTopic>odom</odometryTopic>
+			<odometryFrame>odom</odometryFrame>
+			<odometryRate>20.0</odometryRate>
+			<robotBaseFrame>base_link</robotBaseFrame>
+			<yaw_velocity_p_gain>250</yaw_velocity_p_gain>
+			<publishOdometryTf>0</publishOdometryTf>
+		</plugin>
+	</gazebo> -->
+	<gazebo>
+		<plugin name="imu_controller" filename="libhector_gazebo_ros_imu.so">
+			<robotNamespace>$(arg robot_namespace)</robotNamespace>
+			<updateRate>50.0</updateRate>
+			<bodyName>base_link</bodyName>
+			<topicName>imu/data</topicName>
+			<accelDrift>0.005 0.005 0.005</accelDrift>
+			<accelGaussianNoise>0.005 0.005 0.005</accelGaussianNoise>
+			<rateDrift>0.005 0.005 0.005 </rateDrift>
+			<rateGaussianNoise>0.005 0.005 0.005 </rateGaussianNoise>
+			<headingDrift>0.005</headingDrift>
+			<headingGaussianNoise>0.005</headingGaussianNoise>
+		</plugin>
+	</gazebo>
 </robot>

File: src/carbon_description/urdf/wheel.xacro (robot description, xacro)
@@ -23,10 +23,10 @@
 		</link>
 		<gazebo reference="${wheel_prefix}_wheel_link">
-			<mu1 value="100" />
-			<mu2 value="200" />
+			<mu1 value="0.9" />
+			<mu2 value="0.9" />
 			<kp value="10000000.0" />
 			<kd value="1.0" />
 			<maxVel value="1.0" />
-			<fdir1 value="1 0 0"/>
+			<fdir1 value="0 1 0"/>
 		</gazebo>
 		<joint name="${wheel_prefix}_wheel" type="continuous">
@@ -43,5 +43,5 @@
 			</actuator>
 			<joint name="${wheel_prefix}_wheel">
-				<hardwareInterface>EffortJointInterface</hardwareInterface>
+				<hardwareInterface>hardware_interface/EffortJointInterface</hardwareInterface>
 			</joint>
 		</transmission>

Commit message: urdf

File: src/carbon_description/urdf/carbon.urdf.xacro (robot description, xacro)
@@ -48,4 +48,18 @@
 		</visual>
 	</link>
+	<link name="camera_link">
+                <visual name='camera_box'>
+                        <origin xyz="0 0 0" rpy="0 0 0"/>
+                        <geometry>
+                                <box size="0.05 0.05 0.05"/>
+                        </geometry>
+                        <material name="green"/>
+                </visual>
+		<inertial>
+                        <mass value="${0.005}" />
+                        <origin xyz="0 0 0" rpy=" 0 0 0"/>
+                        <xacro:box_inertia m="${0.005}" x="${0.05}" y="${0.05}" z="${0.05}" />
+                </inertial>
+        </link>
 	<gazebo reference="imu_link">
   	</gazebo>
@@ -66,4 +80,9 @@
 		<origin xyz="0 0 0" rpy="0 0 0"/>
 	</joint>
+	<joint name="base_to_camera" type="fixed">
+                <parent link="base_link"/>
+                <child link="camera_link"/>
+                <origin xyz="0.0 0.0 0.6" rpy="0.0 0.0 0.0" />
+        </joint>
 	<xacro:create_wheel wheel_prefix="left_front">
 		<origin xyz="${track} ${wheelbase/2} ${wheel_vertical_offset}" rpy="0 0 0" />
@@ -89,46 +108,4 @@
 		</plugin>
 	</gazebo>
-	<!-- <gazebo>
-		<plugin name="diff_drive_6w" filename="libdiffdrive_plugin_6w.so">
-			<robotNamespace>$(arg robot_namespace)</robotNamespace>
-			<topicName>/carbon_velocity_controller/cmd_vel</topicName>
-			<frontLeftJoint>left_front_wheel</frontLeftJoint>
-			<midLeftJoint>left_mid_wheel</midLeftJoint>
-			<rearLeftJoint>left_rear_wheel</rearLeftJoint>
-			<frontRightJoint>right_front_wheel</frontRightJoint>
-			<midRightJoint>right_mid_wheel</midRightJoint>
-			<rearRightJoint>right_rear_wheel</rearRightJoint>
-			<wheelSeparation>0.58</wheelSeparation>
-			<wheelDiameter>0.18</wheelDiameter>
-			<torque>50000</torque>
-		</plugin>
-	</gazebo> -->
-	<!-- <gazebo>
-		<plugin name="diffdrive_plugin_multiwheel" filename="libdiffdrive_plugin_multi_wheel.so">
-			<alwaysOn>true</alwaysOn>
-			<updateRate>25.0</updateRate>
-			<leftJoints>left_front_wheel left_mid_wheel left_rear_wheel</leftJoints>
-			<rightJoints>right_front_wheel right_mid_wheel right_rear_wheel</rightJoints>
-			<wheelSeparation>${wheelbase}</wheelSeparation>
-			<wheelDiameter>${wheel_radius*2}</wheelDiameter>
-			<torque>50000</torque>
-			<robotNamespace>/</robotNamespace>
-			<robotBaseFrame>base_link</robotBaseFrame>
-			<commandTopic>/cmd_vel_raw</commandTopic>
-			<publishOdometryTf>0</publishOdometryTf>
-			<publishOdometryMsg>1</publishOdometryMsg>
-		</plugin>
-	</gazebo> -->
-	<!-- <gazebo>
-		<plugin name="force_based_move_controller" filename="libgazebo_ros_force_based_move.so">
-			<commandTopic>/carbon_velocity_controller/cmd_vel</commandTopic>
-			<odometryTopic>odom</odometryTopic>
-			<odometryFrame>odom</odometryFrame>
-			<odometryRate>20.0</odometryRate>
-			<robotBaseFrame>base_link</robotBaseFrame>
-			<yaw_velocity_p_gain>250</yaw_velocity_p_gain>
-			<publishOdometryTf>0</publishOdometryTf>
-		</plugin>
-	</gazebo> -->
 	<gazebo>
 		<plugin name="imu_controller" filename="libhector_gazebo_ros_imu.so">
@@ -145,3 +122,28 @@
 		</plugin>
 	</gazebo>
+	<plugin name="camera_plugin" filename="libgazebo_ros_openni_kinect.so">
+		<baseline>0.2</baseline>
+		<alwaysOn>true</alwaysOn>
+		<!-- Keep this zero, update_rate in the parent <sensor> tag
+		will control the frame rate. -->
+		<updateRate>0.0</updateRate>
+		<cameraName>camera_ir</cameraName>
+		<imageTopicName>/camera/depth/image_raw</imageTopicName>
+		<cameraInfoTopicName>/camera/depth/camera_info</cameraInfoTopicName>
+		<depthImageTopicName>/camera/depth/image_raw</depthImageTopicName>
+		<depthImageInfoTopicName>/camera/depth/camera_info</depthImageInfoTopicName>
+		<pointCloudTopicName>/camera/depth/points</pointCloudTopicName>
+		<frameName>camera_link</frameName>
+		<pointCloudCutoff>0.05</pointCloudCutoff>
+		<distortionK1>0</distortionK1>
+		<distortionK2>0</distortionK2>
+		<distortionK3>0</distortionK3>
+		<distortionT1>0</distortionT1>
+		<distortionT2>0</distortionT2>
+		<CxPrime>0</CxPrime>
+		<Cx>0</Cx>
+		<Cy>0</Cy>
+		<focalLength>0</focalLength>
+		<hackBaseline>0</hackBaseline>
+	</plugin>
 </robot>

Commit message: gazebo working with kinect

File: src/carbon_description/urdf/carbon.urdf.xacro (robot description, xacro)
@@ -14,4 +14,10 @@
 	<xacro:property name="wheel_vertical_offset" value="0.0" />
 	<xacro:arg name="robot_namespace" default="/" />
+   	<xacro:property name="cal_kinect_roll" value="0.0" />
+	<xacro:property name="cal_kinect_pitch" value="0.0" />
+	<xacro:property name="cal_kinect_yaw" value="0.0" />
+	<xacro:property name="cal_kinect_x" value="0.0" />
+	<xacro:property name="cal_kinect_y" value="0.0" />
+	<xacro:property name="cal_kinect_z" value="0.0" />
 	<xacro:include filename="$(find carbon_description)/urdf/macros.xacro" />
 	<xacro:include filename="$(find carbon_description)/urdf/wheel.xacro" />
@@ -85,4 +91,8 @@
                 <origin xyz="0.0 0.0 0.6" rpy="0.0 0.0 0.0" />
         </joint>
+	 <xacro:include filename="$(find carbon_description)/urdf/kinect2.urdf.xacro" />
+	 <xacro:kinect2_v0 name="kinect_mount" parent="camera_link" >
+	 	<origin xyz="0.0 0 0.0" rpy="0 0 0" />
+	 </xacro:kinect2_v0>
 	<xacro:create_wheel wheel_prefix="left_front">
 		<origin xyz="${track} ${wheelbase/2} ${wheel_vertical_offset}" rpy="0 0 0" />
@@ -122,28 +132,3 @@
 		</plugin>
 	</gazebo>
-	<plugin name="camera_plugin" filename="libgazebo_ros_openni_kinect.so">
-		<baseline>0.2</baseline>
-		<alwaysOn>true</alwaysOn>
-		<!-- Keep this zero, update_rate in the parent <sensor> tag
-		will control the frame rate. -->
-		<updateRate>0.0</updateRate>
-		<cameraName>camera_ir</cameraName>
-		<imageTopicName>/camera/depth/image_raw</imageTopicName>
-		<cameraInfoTopicName>/camera/depth/camera_info</cameraInfoTopicName>
-		<depthImageTopicName>/camera/depth/image_raw</depthImageTopicName>
-		<depthImageInfoTopicName>/camera/depth/camera_info</depthImageInfoTopicName>
-		<pointCloudTopicName>/camera/depth/points</pointCloudTopicName>
-		<frameName>camera_link</frameName>
-		<pointCloudCutoff>0.05</pointCloudCutoff>
-		<distortionK1>0</distortionK1>
-		<distortionK2>0</distortionK2>
-		<distortionK3>0</distortionK3>
-		<distortionT1>0</distortionT1>
-		<distortionT2>0</distortionT2>
-		<CxPrime>0</CxPrime>
-		<Cx>0</Cx>
-		<Cy>0</Cy>
-		<focalLength>0</focalLength>
-		<hackBaseline>0</hackBaseline>
-	</plugin>
 </robot>
